File: Garage_PCB.brd (EAGLE design)
At the start: 35.6 x 39.4 mm, 20 parts, among them Q1 MOSFET-NCHANNEL_THRMTO-220-TH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

Commit message: Removed MOSFET inline resistors
The garage door button needs to have a direct connection from power
(btn_h) to ground (btn_l) in order to open or close the garage door.
The high side resistor kept this from happening.  I am not sure what I
was thinking with the low side 'pull down'.  This was just a weird
resistor connecting a groundplane on the opener to a ground plane on my
board.

I also renamed a few of the connection labels on the backside to be
correct.  The btn_p and btn_n were backwards and this was causing the
opener to not work.  The range finders also need to have different
labels so that the user knows which one is connected for configuring the
app/Spark Core.
Parts:
- removed R2: 1K, SparkFun-Resistors:0603-RES
- removed R5: 10K, SparkFun-Resistors:0603-RES
Connections:
- removed net BTN_L: JP4.2, Q1.OUT, R5.2
- removed net N$17: Q1.GND, R2.1
- net BTN_H: now also Q1.GND; no longer R2.2
- net GND: now also JP4.2, Q1.OUT; no longer R5.1
Routing:
- net BTN_L: track 32.6 -> 0.00 mm
- net BTN_H: track 23.1 -> 28.3 mm
- net N$17: track 3.47 -> 0.00 mm
Other:
- board text added: "RNG2_I"
Changed lines of the file:
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@@
 <text x="31.623" y="22.352" size="0.8128" layer="22" font="vector" ratio="15" rot="MR270">GND</text>
 <text x="31.496" y="18.542" size="0.8128" layer="22" font="vector" ratio="15" rot="MR270">5V</text>
-<text x="31.496" y="32.004" size="0.8128" layer="22" font="vector" ratio="15" rot="MR270">BTN_P</text>
-<text x="31.496" y="27.178" size="0.8128" layer="22" font="vector" ratio="15" rot="MR270">BTN_N</text>
+<text x="31.496" y="27.004" size="0.8128" layer="22" font="vector" ratio="15" rot="MR270">BTN_P</text>
+<text x="31.496" y="32.178" size="0.8128" layer="22" font="vector" ratio="15" rot="MR270">BTN_N</text>
 <text x="5.207" y="10.287" size="0.8128" layer="22" font="vector" ratio="15" rot="MR270">LED_O</text>
 <text x="5.207" y="18.923" size="0.8128" layer="22" font="vector" ratio="15" rot="MR270">RNG_I</text>
 <text x="31.623" y="10.922" size="0.8128" layer="22" font="vector" ratio="15" rot="MR270">SW_COM</text>
 <text x="31.623" y="14.859" size="0.8128" layer="22" font="vector" ratio="15" rot="MR270">SW_NO</text>
-<text x="5.207" y="23.749" size="0.8128" layer="22" font="vector" ratio="15" rot="MR270">RNG_I</text>
+<text x="5.207" y="23.749" size="0.8128" layer="22" font="vector" ratio="15" rot="MR270">RNG2_I</text>
 <text x="13.97" y="3.81" size="0.8128" layer="21" font="vector" ratio="15">Designed by
 Mike Loptien</text>
@@
 <attribute name="VALUE" x="25.273" y="26.924" size="0.4064" layer="27" font="vector" rot="R90"/>
 </element>
-<element name="R2" library="SparkFun-Resistors" package="0603-RES" value="1K" x="17.78" y="33.02" rot="R90"/>
 <element name="JP5" library="SparkFun-Connectors" package="SCREWTERMINAL-3.5MM-2" value="M023.5MM" x="33.02" y="9.271" rot="R90"/>
 <element name="R3" library="SparkFun-Resistors" package="0603-RES" value="10K" x="29.718" y="11.811" rot="MR90"/>
@@
 <element name="FRAME2" library="SparkFun-Aesthetics" package="CREATIVE_COMMONS" value="FRAME-LETTER" x="-77.47" y="-12.7"/>
 <element name="JP1" library="SparkFun-Connectors" package="SCREWTERMINAL-3.5MM-2" value="M023.5MM" x="32.893" y="17.399" rot="R90"/>
-<element name="R5" library="SparkFun-Resistors" package="0603-RES" value="10K" x="12.48" y="29.52" rot="MR270"/>
 </elements>
 <signals>
@@
 <via x="16.51" y="19.05" extent="1-16" drill="0.508" shape="square"/>
 <wire x1="16.51" y1="19.05" x2="15.24" y2="17.78" width="0.6096" layer="1"/>
-<contactref element="R5" pad="1"/>
+<contactref element="Q1" pad="OUT"/>
+<contactref element="JP4" pad="2"/>
 </signal>
 <signal name="5V">
@@
 <contactref element="JP3" pad="1"/>
 </signal>
-<signal name="N$17">
-<contactref element="Q1" pad="GND"/>
-<contactref element="R2" pad="1"/>
-<wire x1="17.78" y1="32.17" x2="17.78" y2="28.702" width="0.6096" layer="1"/>
-</signal>
 <signal name="RD_SW_I">
 <contactref element="JP5" pad="2"/>
@@
 <signal name="BTN_H">
 <contactref element="JP4" pad="1"/>
-<contactref element="R2" pad="2"/>
 <wire x1="32.893" y1="25.654" x2="32.766" y2="25.654" width="0.6096" layer="1"/>
 <wire x1="32.766" y1="25.654" x2="29.21" y2="29.21" width="0.6096" layer="1"/>
 <wire x1="29.21" y1="29.21" x2="29.21" y2="34.29" width="0.6096" layer="1"/>
 <wire x1="29.21" y1="34.29" x2="27.94" y2="35.56" width="0.6096" layer="1"/>
-<wire x1="17.78" y1="33.87" x2="17.78" y2="34.29" width="0.6096" layer="1"/>
 <wire x1="17.78" y1="34.29" x2="19.05" y2="35.56" width="0.6096" layer="1"/>
 <wire x1="19.05" y1="35.56" x2="27.94" y2="35.56" width="0.6096" layer="1"/>
-</signal>
-<signal name="BTN_L">
-<contactref element="JP4" pad="2"/>
-<contactref element="Q1" pad="OUT"/>
-<wire x1="32.893" y1="29.154" x2="32.893" y2="33.147" width="0.6096" layer="1"/>
-<wire x1="32.893" y1="33.147" x2="29.21" y2="36.83" width="0.6096" layer="1"/>
-<wire x1="29.21" y1="36.83" x2="17.78" y2="36.83" width="0.6096" layer="1"/>
-<wire x1="17.78" y1="36.83" x2="15.24" y2="34.29" width="0.6096" layer="1"/>
-<wire x1="15.24" y1="34.29" x2="15.24" y2="28.702" width="0.6096" layer="1"/>
-<contactref element="R5" pad="2"/>
-<wire x1="12.48" y1="28.67" x2="15.208" y2="28.67" width="0.6096" layer="16"/>
-<wire x1="15.208" y1="28.67" x2="15.24" y2="28.702" width="0.6096" layer="16"/>
+<contactref element="Q1" pad="GND"/>
+<wire x1="17.78" y1="34.29" x2="17.78" y2="28.702" width="0.6096" layer="1"/>
 </signal>
 </signals>
